File: redox/pcb/rev1.0/kicad_files/redox_rev1.sch (KiCad schematic (older format))
At the start: 76 parts, among them K0 KEYSW, K1 KEYSW, K10 KEYSW, K11 KEYSW, K12 KEYSW, K13 KEYSW, K14 KEYSW, K15 KEYSW, K16 KEYSW, K2 KEYSW, K20 KEYSW, K21 KEYSW, K22 KEYSW, K23 KEYSW, K24 KEYSW, K25 KEYSW, K26 KEYSW, K3 KEYSW, K30 KEYSW, K31 KEYSW, K32 KEYSW, K33 KEYSW, K34 KEYSW, K35 KEYSW, K36 KEYSW, K4 KEYSW, K40 KEYSW, K41 KEYSW, K42 KEYSW, K43 KEYSW, K44 KEYSW, K45 KEYSW, K46 KEYSW, K5 KEYSW, K6 KEYSW, U1 ProMicro

Commit message: Update to reversible kailh hotswap
Parts:
- removed RGB_STRIP1: Conn_01x03, Pin_Headers:Pin_Header_Straight_1x03_Pitch2.54mm, symbol Conn_01x03
- removed U1: ProMicro, Keebio-Parts:ArduinoProMicro, symbol ProMicro
- added BP1: BlackPill2, reversable_hotswap:BlackPill, symbol STM32BlackPill2:BlackPill2
- D0, D1, D10, D11, D12, D13, D14, D15, D16, D2, D20, D21, D22, D23, D24, D25, D26, D3, D30, D31, D32, D33, D34, D35, D36, D4, D40, D41, D42, D43, D44, D45, D46, D5, D6: symbol D -> Device:D
- K0, K10, K20, K30, K44: footprint Keebio-Parts:Hybrid_PCB_100H_Dual_hole-nosilk -> reversable_hotswap:MXOnly-1.25U-Hotswap; symbol KEYSW -> keyboard_parts:KEYSW
- K1, K11, K12, K14, K15, K2, K21, K22, K24, K25, K26, K31, K32, K33, K34, K35, K36, K4, K40, K41, K42, K43, K5, K6: footprint Keebio-Parts:Hybrid_PCB_100H_Dual_hole-nosilk -> reversable_hotswap:MXOnly-1U-Hotswap; symbol KEYSW -> keyboard_parts:KEYSW
- K13, K23, K3: footprint Keebio-Parts:Hybrid_PCB_100H_Dual_hole-nosilk -> reversable_hotswap:MXOnly-1U-Hotswap-Small; symbol KEYSW -> keyboard_parts:KEYSW
- K16, K45, K46: footprint Keebio-Parts:Hybrid_PCB_100H_Dual_hole-nosilk -> reversable_hotswap:MXOnly-1.5U-Hotswap; symbol KEYSW -> keyboard_parts:KEYSW
- R1, R2: symbol R -> Device:R
- RST_SW1: symbol SW_PUSH -> keyboard_parts:SW_PUSH
- TRRS1: symbol Audio-Jack-4 -> redox_rev1-rescue:Audio-Jack-4
Connections:
- net labels removed: rgb_data
- wire segments 69 -> 133
- no-connect marks 4 -> 0
Other:
- moved on the sheet: TRRS1

Commit message: Finish routing and top silkscreen
Parts:
- BP1: symbol STM32BlackPill2:BlackPill2 -> redox_rev1-rescue:BlackPill2-STM32BlackPill2
Connections:
- net VCC: no longer BP1.21 (3.3V)
- net col3: now also BP1.36 (A8); no longer BP1.4 (B10)
- net col4: now also BP1.4 (B10); no longer BP1.5 (B2)
- net col5: now also BP1.5 (B2); no longer BP1.6 (B1)
- net col6: now also BP1.6 (B1); no longer BP1.7 (B0)
- net row0: now also BP1.32 (A12); no longer BP1.40 (B12)
- net row1: now also BP1.29 (B4); no longer BP1.34 (A10)
Other:
- moved on the sheet: D0, D1, D10, D11, D12, D13, D14, D15, D16, D2, D20, D21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
