File: redox/pcb/rev1.0/kicad_files/redox_hotswap_led.kicad_pcb (KiCad board)
At the start: 2 copper layers, 162.2 x 126.5 mm, 106 parts, among them K0 SW_Push_LED, K1 SW_Push_LED, K10 SW_Push_LED, K11 SW_Push_LED, K12 SW_Push_LED, K13 SW_Push_LED, K14 SW_Push_LED, K15 SW_Push_LED, K16 SW_Push_LED, K2 SW_Push_LED, K20 SW_Push_LED, K21 SW_Push_LED, K22 SW_Push_LED, K23 SW_Push_LED, K24 SW_Push_LED, K25 SW_Push_LED, K26 SW_Push_LED, K3 SW_Push_LED, K30 SW_Push_LED, K31 SW_Push_LED, K32 SW_Push_LED, K33 SW_Push_LED, K34 SW_Push_LED, K35 SW_Push_LED, K36 SW_Push_LED, K4 SW_Push_LED, K40 SW_Push_LED, K41 SW_Push_LED, K42 SW_Push_LED, K43 SW_Push_LED, K44 SW_Push_LED, K45 SW_Push_LED, K46 SW_Push_LED, K5 SW_Push_LED, K6 SW_Push_LED, Q1 BC848, Q10 BC848, Q11 BC848, Q12 BC848, Q2 BC848, Q3 BC848, Q4 BC848, Q5 BC848, Q6 BC848, Q7 BC848, Q8 BC848, Q9 BC848

Commit message: Complete routing and PCB
Parts:
- turned Q11 to 90 degrees
Routing:
- net Net-(Q11-Pad1): track 7.66 -> 4.47 mm
- net Net-(Q3-Pad1): track 4.77 -> 7.53 mm
- net GND: track 31.9 -> 33.9 mm, vias 159 -> 158
- net Net-(Q10-Pad1): track 4.05 -> 5.97 mm
- net Net-(Q1-Pad1): track 5.40 -> 6.56 mm
- net Net-(Q8-Pad1): track 5.61 -> 6.68 mm
- net Net-(Q9-Pad3): track 7.52 -> 6.58 mm
- net Net-(K40-Pad4): track 141.3 -> 140.5 mm
- net VCC: track 239.6 -> 238.9 mm
- net Net-(Q4-Pad1): track 5.58 -> 6.13 mm
- net Net-(K30-Pad4): track 174.4 -> 175.0 mm
- net Net-(K10-Pad4): track 156.1 -> 156.6 mm
Other:
- board text removed: "designed by Mattia Dal Ben (https://github.com/mattdibi)"
