File: redox/pcb/rev1.0/kicad_files/redox_hotswap_led.sch (KiCad schematic (older format))
At the start: 106 parts, among them K0 SW_Push_LED, K1 SW_Push_LED, K10 SW_Push_LED, K11 SW_Push_LED, K12 SW_Push_LED, K13 SW_Push_LED, K14 SW_Push_LED, K15 SW_Push_LED, K16 SW_Push_LED, K2 SW_Push_LED, K20 SW_Push_LED, K21 SW_Push_LED, K22 SW_Push_LED, K23 SW_Push_LED, K24 SW_Push_LED, K25 SW_Push_LED, K26 SW_Push_LED, K3 SW_Push_LED, K30 SW_Push_LED, K31 SW_Push_LED, K32 SW_Push_LED, K33 SW_Push_LED, K34 SW_Push_LED, K35 SW_Push_LED, K36 SW_Push_LED, K4 SW_Push_LED, K40 SW_Push_LED, K41 SW_Push_LED, K42 SW_Push_LED, K43 SW_Push_LED, K44 SW_Push_LED, K45 SW_Push_LED, K46 SW_Push_LED, K5 SW_Push_LED, K6 SW_Push_LED, Q1 BC848, Q10 BC848, Q11 BC848, Q12 BC848, Q2 BC848, Q3 BC848, Q4 BC848, Q5 BC848, Q6 BC848, Q7 BC848, Q8 BC848, Q9 BC848

Commit message: ?
Parts:
- BP1: symbol STM32BlackPill2:BlackPill2 -> redox_hotswap_led-rescue:BlackPill2-STM32BlackPill2
Changed lines of the file:
@@
 $EndComp
 $Comp
-L STM32BlackPill2:BlackPill2 BP1
+L redox_hotswap_led-rescue:BlackPill2-STM32BlackPill2 BP1
 U 1 1 5E52B74E
 P 2250 1750
